Commit message: fix: remove xacro pi redefinition

File: src/pick_and_place/urdf/arm.urdf.xacro (robot description, xacro)
@@ -13,5 +13,4 @@
   <xacro:property name="finger_length" value="0.06"/>
   <xacro:property name="finger_width" value="0.01"/>
-  <xacro:property name="pi" value="3.14159265359"/>
   <!-- ================= INERTIA MACROS ================= -->
   <xacro:macro name="cylinder_inertia" params="mass length radius">
